File: Ethan James/MyFirstKiCAD/_autosave-MyFirstKiCAD.kicad_sch (KiCad schematic)
At the start: 3 parts, among them SW1 SW_Push

Commit message: commit 1
Parts:
- removed D1: LED, symbol Device:LED
- removed R1: R_US, symbol Device:R_US
- added BT1: Battery_Cell, FS_3_Global_Footprint_Library:MS621FE-FL11E_SEC, symbol Device:Battery_Cell
- added D1: D, LED_SMD:LED_0805_2012Metric_Pad1.15x1.40mm_HandSolder, symbol Device:D
- added R1: R, Resistor_SMD:R_0805_2012Metric_Pad1.20x1.40mm_HandSolder, symbol Device:R
- SW1: footprint (none) -> Button_Switch_SMD:SW_MEC_5GSH9
Connections:
- net at SW1.1: now also R1.1
- net at SW1.2: now also D1.2 (A)
- new net: BT1.1 (+), R1.2
- new net: BT1.2 (-), D1.1 (K)
Changed lines of the file:
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@@
 	(wire
 		(pts
-			(xy 59.69 39.37) (xy 64.77 39.37)
+			(xy 57.15 39.37) (xy 64.77 39.37)
 		)
 		(stroke
@@
 	(wire
 		(pts
-			(xy 41.91 39.37) (xy 46.99 39.37)
+			(xy 41.91 39.37) (xy 49.53 39.37)
 		)
 		(stroke
@@
 	)
 	(symbol
-		(lib_id "power:GND")
-		(at 59.69 39.37 0)
+		(lib_id "Device:R")
+		(at 41.91 31.75 0)
 		(unit 1)
 		(exclude_from_sim no)
@@
 		(dnp no)
 		(fields_autoplaced yes)
-		(property "Reference" "#PWR02"
-			(at 59.69 45.72 0)
-			(effects
-				(font
-					(size 1.27 1.27)
-				)
-				(hide yes)
-			)
-		)
-		(property "Value" "GND"
-			(at 59.69 44.45 0)
-			(effects
-				(font
-					(size 1.27 1.27)
-				)
-			)
-		)
-		(property "Footprint" ""
-			(at 59.69 39.37 0)
-			(effects
-				(font
-					(size 1.27 1.27)
-				)
-				(hide yes)
-			)
-		)
-		(property "Datasheet" ""
-			(at 59.69 39.37 0)
-			(effects
-				(font
-					(size 1.27 1.27)
-				)
-				(hide yes)
-			)
-		)
-		(property "Description" "Power symbol creates a global label with name \"GND\" , ground"
-			(at 59.69 39.37 0)
+		(property "Reference" "R1"
+			(at 44.45 30.4799 0)
+			(effects
+				(font
+					(size 1.27 1.27)
+				)
+				(justify left)
+			)
+		)
+		(property "Value" "R"
+			(at 44.45 33.0199 0)
+			(effects
+				(font
+					(size 1.27 1.27)
+				)
+				(justify left)
+			)
+		)
+		(property "Footprint" "Resistor_SMD:R_0805_2012Metric_Pad1.20x1.40mm_HandSolder"
+			(at 40.132 31.75 90)
+			(effects
+				(font
+					(size 1.27 1.27)
+				)
+				(hide yes)
+			)
+		)
+		(property "Datasheet" "~"
+			(at 41.91 31.75 0)
+			(effects
+				(font
+					(size 1.27 1.27)
+				)
+				(hide yes)
+			)
+		)
+		(property "Description" "Resistor"
+			(at 41.91 31.75 0)
 			(effects
 				(font
@@
 		)
 		(pin "1"
+		)
+		(pin "2"
 		)
 		(instances
 			(project ""
 				(path "/9bb8b0c9-2404-456a-897c-7e797b4600f0"
-					(reference "#PWR02")
+					(reference "R1")
 					(unit 1)
 				)
@@
 			)
 		)
-		(property "Footprint" ""
+		(property "Footprint" "Button_Switch_SMD:SW_MEC_5GSH9"
 			(at 53.34 20.32 0)
 			(effects
@@
 	)
 	(symbol
-		(lib_id "Device:LED")
+		(lib_id "Device:D")
 		(at 64.77 31.75 90)
 		(unit 1)
@@
 		(fields_autoplaced yes)
 		(property "Reference" "D1"
-			(at 68.58 32.0674 90)
+			(at 67.31 30.4799 90)
 			(effects
 				(font
@@
 			)
 		)
-		(property "Value" "LED"
-			(at 68.58 34.6074 90)
+		(property "Value" "D"
+			(at 67.31 33.0199 90)
 			(effects
 				(font
@@
 			)
 		)
-		(property "Footprint" ""
+		(property "Footprint" "LED_SMD:LED_0805_2012Metric_Pad1.15x1.40mm_HandSolder"
 			(at 64.77 31.75 0)
 			(effects
@@
 			)
 		)
-		(property "Description" "Light emitting diode"
-			(at 64.77 31.75 0)
-			(effects
-				(font
-					(size 1.27 1.27)
-				)
-				(hide yes)
-			)
+		(property "Description" "Diode"
+			(at 64.77 31.75 0)
+			(effects
+				(font
+					(size 1.27 1.27)
+				)
+				(hide yes)
+			)
+		)
+		(property "Sim.Device" "D"
+			(at 64.77 31.75 0)
+			(effects
+				(font
+					(size 1.27 1.27)
+				)
+				(hide yes)
+			)
+		)
+		(property "Sim.Pins" "1=K 2=A"
+			(at 64.77 31.75 0)
+			(effects
+				(font
+					(size 1.27 1.27)
+				)
+				(hide yes)
+			)
+		)
+		(pin "2"
 		)
 		(pin "1"
-		)
-		(pin "2"
 		)
 		(instances
@@
 	)
 	(symbol
-		(lib_id "power:VSS")
-		(at 46.99 39.37 180)
+		(lib_id "Device:Battery_Cell")
+		(at 54.61 39.37 90)
 		(unit 1)
 		(exclude_from_sim no)
@@
 		(dnp no)
 		(fields_autoplaced yes)
-		(property "Reference" "#PWR01"
-			(at 46.99 35.56 0)
-			(effects
-				(font
-					(size 1.27 1.27)
-				)
-				(hide yes)
-			)
-		)
-		(property "Value" "VSS"
-			(at 46.99 44.45 0)
-			(effects
-				(font
-					(size 1.27 1.27)
-				)
-			)
-		)
-		(property "Footprint" ""
-			(at 46.99 39.37 0)
-			(effects
-				(font
-					(size 1.27 1.27)
-				)
-				(hide yes)
-			)
-		)
-		(property "Datasheet" ""
-			(at 46.99 39.37 0)
-			(effects
-				(font
-					(size 1.27 1.27)
-				)
-				(hide yes)
-			)
-		)
-		(property "Description" "Power symbol creates a global label with name \"VSS\""
-			(at 46.99 39.37 0)
+		(property "Reference" "BT1"
+			(at 52.7685 31.75 90)
+			(effects
+				(font
+					(size 1.27 1.27)
+				)
+			)
+		)
+		(property "Value" "Battery_Cell"
+			(at 52.7685 34.29 90)
+			(effects
+				(font
+					(size 1.27 1.27)
+				)
+			)
+		)
+		(property "Footprint" "FS_3_Global_Footprint_Library:MS621FE-FL11E_SEC"
+			(at 53.086 39.37 90)
+			(effects
+				(font
+					(size 1.27 1.27)
+				)
+				(hide yes)
+			)
+		)
+		(property "Datasheet" "~"
+			(at 53.086 39.37 90)
+			(effects
+				(font
+					(size 1.27 1.27)
+				)
+				(hide yes)
+			)
+		)
+		(property "Description" "Single-cell battery"
+			(at 54.61 39.37 0)
 			(effects
 				(font
@@
 		)
 		(pin "1"
+		)
+		(pin "2"
 		)
 		(instances
 			(project ""
 				(path "/9bb8b0c9-2404-456a-897c-7e797b4600f0"
-					(reference "#PWR01")
+					(reference "BT1")
 					(unit 1)
 				)
-			)
-		)
-	)
-	(symbol
-		(lib_id "Device:R_US")
-		(at 41.91 31.75 0)
-		(unit 1)
-		(exclude_from_sim no)
-		(in_bom yes)
-		(on_board yes)
-		(dnp no)
-		(fields_autoplaced yes)
-		(property "Reference" "R1"
-			(at 44.45 30.4799 0)
-			(effects
-				(font
-					(size 1.27 1.27)
-				)
-				(justify left)
-			)
-		)
-		(property "Value" "R_US"
-			(at 44.45 33.0199 0)
-			(effects
-				(font
-					(size 1.27 1.27)
-				)
-				(justify left)
-			)
-		)
-		(property "Footprint" ""
-			(at 42.926 32.004 90)
-			(effects
-				(font
-					(size 1.27 1.27)
-				)
-				(hide yes)
-			)
-		)
-		(property "Datasheet" "~"
-			(at 41.91 31.75 0)
-			(effects
-				(font
-					(size 1.27 1.27)
-				)
-				(hide yes)
-			)
-		)
-		(property "Description" "Resistor, US symbol"
-			(at 41.91 31.75 0)
-			(effects
-				(font
-					(size 1.27 1.27)
-				)
-				(hide yes)
-			)
-		)
-		(pin "1"
-		)
-		(pin "2"
-		)
-		(instances
-			(project ""
-				(path "/9bb8b0c9-2404-456a-897c-7e797b4600f0"
-					(reference "R1")
-					(unit 1)
-				)
