File: Nathaniel Platt/KiCad first project/KiCad first project.kicad_sch (KiCad schematic)
At the start: 0 parts

Commit message: pcb demoing
Parts:
- added D1: D, Diode_SMD:D_0805_2012Metric_Pad1.15x1.40mm_HandSolder, symbol Device:D
- added R1: R, Resistor_SMD:R_0805_2012Metric_Pad1.20x1.40mm_HandSolder, symbol Device:R
Connections:
- new net: D1.2 (A), R1.2
- new net Battery +: R1.1
- new net Battery -: D1.1 (K)
Other:
- added sheet Untitled Sheet (untitled.kicad_sch)
