File: Ruandy Salazar/LED Board/LED Board.kicad_sch (KiCad schematic)
At the start: 3 parts

Commit message: Intro Project Changes
Peripheral Board
Parts:
- BT1: footprint Battery:BatteryHolder_Seiko_MS621F -> FS_3_Global_Footprint_Library:MS621FE-FL11E_SEC
Changed lines of the file:
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@@
 			)
 		)
-		(property "Footprint" "Battery:BatteryHolder_Seiko_MS621F"
+		(property "Footprint" "FS_3_Global_Footprint_Library:MS621FE-FL11E_SEC"
 			(at 57.15 92.456 90)
 			(effects
