File: Ruandy Salazar/F3 peripheral boards/F3 peripheral boards.kicad_sch (KiCad schematic)
At the start: 29 parts, among them J1 Hall Effect Sensor, J2 105313-1108, J3 Potentiometer, J4 Strain Gauge

Commit message: Peripheral Board Schematic
Parts:
- added C5: 100nF, symbol Device:C
- added R10: ~, symbol Device:R_US
- added R11: 0.64, symbol Device:R_US
- added TP9: VrefBG, symbol Connector:TestPoint
- added U1: INA125U, symbol New_Library:INA125U
Connections:
- net +3V3: now also C5.1, U1.1 (V+), U1.2 (*SLEEP)
- net GND: now also C5.2, U1.12 (VREFCOM), U1.3 (V-)
- net Strain: now also U1.10 (VO), U1.11 (SENSE)
- net Vin+: now reaches J4.2 (Pin_1), R9.1
- net Vin-: now reaches R7.2, R8.1
- new net RG1: R10.1, R11.1, U1.8 (RG)
- new net RG2: R10.2, R11.2, U1.9 (RG)
- new net VIN+: U1.6 (VIN+)
- new net VIN-: U1.7 (VIN-)
- new net VrefBG: TP9.1, U1.13 (VREFBG), U1.4 (VREFOUT), U1.5 (IAREF)
Other:
- note added: "Gain Resistor"
- note added: "Wheatstone Bridge"
- moved on the sheet: J4, R7, R8, R9
